Commit message: increased size of marker

File: urdf/chilitag.urdf.xacro (robot description, xacro)
@@ -16,5 +16,5 @@
         <origin xyz="0 0 0" rpy="0 -1.57079632679 0"/>
         <geometry>
-          <mesh filename="package://vigir_ar_alvar_description/meshes/${name}.dae"/>
+          <mesh scale="1 1.66 1.66" filename="package://vigir_ar_alvar_description/meshes/${name}.dae"/>
         </geometry>
       </visual>
@@ -22,5 +22,5 @@
         <origin xyz="0 0 0" rpy="0 0 0"/>
         <geometry>
-          <mesh filename="package://vigir_ar_alvar_description/meshes/${name}.dae"/>
+          <mesh scale="1 1.66 1.66" filename="package://vigir_ar_alvar_description/meshes/${name}.dae"/>
         </geometry>
       </collision>
@@ -40,5 +40,5 @@
         <origin xyz="0 0 0" rpy="0 0 0"/>
         <geometry>
-          <box size="0.05 0.05 0.001" />
+          <box size="0.065 0.065 0.001" />
         </geometry>
       </visual>

Commit message: fixed wrong package name

File: urdf/chilitag.urdf.xacro (robot description, xacro)
@@ -16,5 +16,5 @@
         <origin xyz="0 0 0" rpy="0 -1.57079632679 0"/>
         <geometry>
-          <mesh scale="1 1.66 1.66" filename="package://vigir_ar_alvar_description/meshes/${name}.dae"/>
+          <mesh scale="1 1.66 1.66" filename="package://hector_chilitag_description/meshes/${name}.dae"/>
         </geometry>
       </visual>
@@ -22,5 +22,5 @@
         <origin xyz="0 0 0" rpy="0 0 0"/>
         <geometry>
-          <mesh scale="1 1.66 1.66" filename="package://vigir_ar_alvar_description/meshes/${name}.dae"/>
+          <mesh scale="1 1.66 1.66" filename="package://hector_chilitag_description/meshes/${name}.dae"/>
         </geometry>
       </collision>

Commit message: fixed collision geometry

File: urdf/chilitag.urdf.xacro (robot description, xacro)
@@ -20,5 +20,5 @@
       </visual>
       <collision>
-        <origin xyz="0 0 0" rpy="0 0 0"/>
+        <origin xyz="0 0 0" rpy="0 -1.57079632679 0"/>
         <geometry>
           <mesh scale="1 1.66 1.66" filename="package://hector_chilitag_description/meshes/${name}.dae"/>
@@ -46,5 +46,5 @@
         <origin xyz="0 0 0" rpy="0 0 0"/>
         <geometry>
-          <box size="0.1 0.1 0.0001" />
+          <box size="0.065 0.065 0.001" />
         </geometry>
       </collision>

Commit message: added size parameter

File: urdf/chilitag.urdf.xacro (robot description, xacro)
@@ -1,5 +1,5 @@
 <?xml version="1.0"?>
 <robot xmlns:xacro="http://playerstage.sourceforge.net/gazebo/xmlschema/#interface" name="artag" >
-  <xacro:macro name="artag" params="name parent *origin">
+  <xacro:macro name="artag" params="name size parent *origin">
     <joint name="${name}_joint" type="fixed">
       <xacro:insert_block name="origin" />
@@ -16,5 +16,5 @@
         <origin xyz="0 0 0" rpy="0 -1.57079632679 0"/>
         <geometry>
-          <mesh scale="1 1.66 1.66" filename="package://hector_chilitag_description/meshes/${name}.dae"/>
+          <mesh scale="${size} ${size} ${size}" filename="package://hector_chilitag_description/meshes/${name}.dae"/>
         </geometry>
       </visual>
@@ -22,5 +22,5 @@
         <origin xyz="0 0 0" rpy="0 -1.57079632679 0"/>
         <geometry>
-          <mesh scale="1 1.66 1.66" filename="package://hector_chilitag_description/meshes/${name}.dae"/>
+          <mesh scale="${size} ${size} ${size}" filename="package://hector_chilitag_description/meshes/${name}.dae"/>
         </geometry>
       </collision>
@@ -40,5 +40,5 @@
         <origin xyz="0 0 0" rpy="0 0 0"/>
         <geometry>
-          <box size="0.065 0.065 0.001" />
+          <box size="${size + 0.015} ${size + 0.015} 0.001" />
         </geometry>
       </visual>
@@ -46,5 +46,5 @@
         <origin xyz="0 0 0" rpy="0 0 0"/>
         <geometry>
-          <box size="0.065 0.065 0.001" />
+          <box size="${size + 0.015} ${size + 0.015} 0.001" />
         </geometry>
       </collision>

Commit message: Refactor chilitag macros for more versatile use

File: urdf/chilitag.urdf.xacro (robot description, xacro)
@@ -1,4 +1,28 @@
 <?xml version="1.0"?>
 <robot xmlns:xacro="http://playerstage.sourceforge.net/gazebo/xmlschema/#interface" name="artag" >
+  <xacro:macro name="artag_visual_sized" params="name size *origin">
+    <visual>
+      <xacro:insert_block name="origin" />
+      <geometry>
+        <mesh scale="${size} ${size} ${size}" filename="package://hector_chilitag_description/meshes/${name}.dae"/>
+      </geometry>
+    </visual>
+  </xacro:macro>
+  <xacro:macro name="artag_no_geom" params="name size parent *origin">
+    <joint name="${name}_joint" type="fixed">
+      <xacro:insert_block name="origin" />
+      <parent link="${parent}"/>
+      <child link="${name}_link"/>
+    </joint>
+    <link name="${name}_link">
+    </link>
+    <gazebo reference="${name}_link">
+      <!--
+      <material>artag/${name}</material>
+      <turnGravityOff>false</turnGravityOff>
+      <static>false</static>
+      -->
+    </gazebo>
+  </xacro:macro>
   <xacro:macro name="artag" params="name size parent *origin">
     <joint name="${name}_joint" type="fixed">
@@ -13,4 +37,8 @@
         <inertia  ixx="0.00000001" ixy="0.0"  ixz="0.0"  iyy="0.00000001"  iyz="0.0"  izz="0.00000001" />
       </inertial>
+      <xacro:artag_visual_sized name="${name}" size="${size}">
+        <origin xyz="0 0 0" rpy="0 -1.57079632679 0"/>
+      </xacro:artag_visual_sized>
+      <!--
       <visual>
         <origin xyz="0 0 0" rpy="0 -1.57079632679 0"/>
@@ -19,4 +47,6 @@
         </geometry>
       </visual>
+      -->
+      <!--
       <collision>
         <origin xyz="0 0 0" rpy="0 -1.57079632679 0"/>
@@ -25,28 +55,5 @@
         </geometry>
       </collision>
-    </link>
-     <joint name="${name}_background_joint" type="fixed">
-      <origin xyz="0 0 -0.001" rpy="0 0 0" />
-      <parent link="${name}_link"/>
-      <child link="${name}_background_link"/>
-    </joint>
-    <link name="${name}_background_link">
-      <inertial>
-        <origin xyz="0 0 0" />
-        <mass value="0.01" />
-        <inertia  ixx="0.00000001" ixy="0.0"  ixz="0.0"  iyy="0.00000001"  iyz="0.0"  izz="0.00000001" />
-      </inertial>
-      <visual>
-        <origin xyz="0 0 0" rpy="0 0 0"/>
-        <geometry>
-          <box size="${size + 0.015} ${size + 0.015} 0.001" />
-        </geometry>
-      </visual>
-      <collision>
-        <origin xyz="0 0 0" rpy="0 0 0"/>
-        <geometry>
-          <box size="${size + 0.015} ${size + 0.015} 0.001" />
-        </geometry>
-      </collision>
+      -->
     </link>
     <gazebo reference="${name}_link">
@@ -57,11 +64,4 @@
       -->
     </gazebo>
-    <gazebo reference="${name}_background_link">
-      <material>Gazebo/White</material>
-      <!--
-      <turnGravityOff>false</turnGravityOff>
-      <static>false</static>
-      -->
-    </gazebo>
   </xacro:macro>
 </robot>

Commit message: Rename macro names from artag to chilitag

File: urdf/chilitag.urdf.xacro (robot description, xacro)
@@ -1,5 +1,5 @@
 <?xml version="1.0"?>
-<robot xmlns:xacro="http://playerstage.sourceforge.net/gazebo/xmlschema/#interface" name="artag" >
-  <xacro:macro name="artag_visual_sized" params="name size *origin">
+<robot xmlns:xacro="http://playerstage.sourceforge.net/gazebo/xmlschema/#interface" name="chilitag" >
+  <xacro:macro name="chilitag_visual_sized" params="name size *origin">
     <visual>
       <xacro:insert_block name="origin" />
@@ -9,5 +9,5 @@
     </visual>
   </xacro:macro>
-  <xacro:macro name="artag_no_geom" params="name size parent *origin">
+  <xacro:macro name="chilitag_no_geom" params="name size parent *origin">
     <joint name="${name}_joint" type="fixed">
       <xacro:insert_block name="origin" />
@@ -18,12 +18,7 @@
     </link>
     <gazebo reference="${name}_link">
-      <!--
-      <material>artag/${name}</material>
-      <turnGravityOff>false</turnGravityOff>
-      <static>false</static>
-      -->
     </gazebo>
   </xacro:macro>
-  <xacro:macro name="artag" params="name size parent *origin">
+  <xacro:macro name="chilitag" params="name size parent *origin">
     <joint name="${name}_joint" type="fixed">
       <xacro:insert_block name="origin" />
@@ -37,7 +32,7 @@
         <inertia  ixx="0.00000001" ixy="0.0"  ixz="0.0"  iyy="0.00000001"  iyz="0.0"  izz="0.00000001" />
       </inertial>
-      <xacro:artag_visual_sized name="${name}" size="${size}">
+      <xacro:chilitag_visual_sized name="${name}" size="${size}">
         <origin xyz="0 0 0" rpy="0 -1.57079632679 0"/>
-      </xacro:artag_visual_sized>
+      </xacro:chilitag_visual_sized>
       <!--
       <visual>
@@ -58,9 +53,4 @@
     </link>
     <gazebo reference="${name}_link">
-      <!--
-      <material>artag/${name}</material>
-      <turnGravityOff>false</turnGravityOff>
-      <static>false</static>
-      -->
     </gazebo>
   </xacro:macro>

Commit message: added new chilitag macro with frame exactly like chillitag 3d detector frame

File: urdf/chilitag.urdf.xacro (robot description, xacro)
@@ -55,3 +55,22 @@
     </gazebo>
   </xacro:macro>
+    <xacro:macro name="chilitag3d" params="name size parent *origin">
+    <joint name="${name}_joint" type="fixed">
+      <xacro:insert_block name="origin" />
+      <parent link="${parent}"/>
+      <child link="${name}_link"/>
+    </joint>
+    <link name="${name}_link">
+      <inertial>
+        <origin xyz="0 0 0" />
+        <mass value="0.01" />
+        <inertia  ixx="0.00000001" ixy="0.0"  ixz="0.0"  iyy="0.00000001"  iyz="0.0"  izz="0.00000001" />
+      </inertial>
+      <xacro:chilitag_visual_sized name="${name}" size="${size}">
+        <origin xyz="${size/2} ${size/2} 0" rpy="${-M_PI/2} ${M_PI/2} ${M_PI}"/>
+      </xacro:chilitag_visual_sized>
+    </link>
+    <gazebo reference="${name}_link">
+    </gazebo>
+  </xacro:macro>
 </robot>

Commit message: Added new macro to allow multiple use of same chilitag

File: urdf/chilitag.urdf.xacro (robot description, xacro)
@@ -74,3 +74,22 @@
     </gazebo>
   </xacro:macro>
+  <xacro:macro name="multi_chilitag" params="name size parent *origin">
+    <joint name="${parent}_${name}_joint" type="fixed">
+      <xacro:insert_block name="origin" />
+      <parent link="${parent}"/>
+      <child link="${parent}_${name}_link"/>
+    </joint>
+    <link name="${parent}_${name}_link">
+      <inertial>
+        <origin xyz="0 0 0" />
+        <mass value="0.01" />
+        <inertia  ixx="0.00000001" ixy="0.0"  ixz="0.0"  iyy="0.00000001"  iyz="0.0"  izz="0.00000001" />
+      </inertial>
+      <xacro:chilitag_visual_sized name="${name}" size="${size}">
+        <origin xyz="${size/2} ${size/2} 0" rpy="${-M_PI/2} ${M_PI/2} ${M_PI}"/>
+      </xacro:chilitag_visual_sized>
+    </link>
+    <gazebo reference="${parent}_${name}_link">
+    </gazebo>
+  </xacro:macro>
 </robot>

Commit message: Added chilitag macro to move chilitags so that the origin is on the corner

File: urdf/chilitag.urdf.xacro (robot description, xacro)
@@ -34,4 +34,39 @@
       <xacro:chilitag_visual_sized name="${name}" size="${size}">
         <origin xyz="0 0 0" rpy="0 -1.57079632679 0"/>
+      </xacro:chilitag_visual_sized>
+      <!--
+      <visual>
+        <origin xyz="0 0 0" rpy="0 -1.57079632679 0"/>
+        <geometry>
+          <mesh scale="${size} ${size} ${size}" filename="package://hector_chilitag_description/meshes/${name}.dae"/>
+        </geometry>
+      </visual>
+      -->
+      <!--
+      <collision>
+        <origin xyz="0 0 0" rpy="0 -1.57079632679 0"/>
+        <geometry>
+          <mesh scale="${size} ${size} ${size}" filename="package://hector_chilitag_description/meshes/${name}.dae"/>
+        </geometry>
+      </collision>
+      -->
+    </link>
+    <gazebo reference="${name}_link">
+    </gazebo>
+  </xacro:macro>
+  <xacro:macro name="chilitag_origin_in_corner" params="name size parent *origin">
+    <joint name="${name}_joint" type="fixed">
+      <xacro:insert_block name="origin" />
+      <parent link="${parent}"/>
+      <child link="${name}_link"/>
+    </joint>
+    <link name="${name}_link">
+      <inertial>
+        <origin xyz="${size/2} ${size/2} 0" />
+        <mass value="0.01" />
+        <inertia  ixx="0.00000001" ixy="0.0"  ixz="0.0"  iyy="0.00000001"  iyz="0.0"  izz="0.00000001" />
+      </inertial>
+      <xacro:chilitag_visual_sized name="${name}" size="${size}">
+        <origin xyz="${size/2} ${size/2} 0" rpy="0 -1.57079632679 0"/>
       </xacro:chilitag_visual_sized>
       <!--

Commit message: Created macro for chilitag 4er set

File: urdf/chilitag.urdf.xacro (robot description, xacro)
@@ -70,23 +70,33 @@
         <origin xyz="${size/2} ${size/2} 0" rpy="0 -1.57079632679 0"/>
       </xacro:chilitag_visual_sized>
-      <!--
-      <visual>
-        <origin xyz="0 0 0" rpy="0 -1.57079632679 0"/>
-        <geometry>
-          <mesh scale="${size} ${size} ${size}" filename="package://hector_chilitag_description/meshes/${name}.dae"/>
-        </geometry>
-      </visual>
-      -->
-      <!--
-      <collision>
-        <origin xyz="0 0 0" rpy="0 -1.57079632679 0"/>
-        <geometry>
-          <mesh scale="${size} ${size} ${size}" filename="package://hector_chilitag_description/meshes/${name}.dae"/>
-        </geometry>
-      </collision>
-      -->
     </link>
     <gazebo reference="${name}_link">
     </gazebo>
+  </xacro:macro>
+  <xacro:macro name="chilitag_4_set" params="name_start offset_x offset_y offset_z offset_tag size parent">
+      <xacro:chilitag_origin_in_corner name="chilitag${name_start}" size="${size}" parent="${parent}">
+        <origin xyz="${offset_x}
+                     ${offset_y}
+                     ${offset_z}"
+                rpy="0 0 0"/>
+      </xacro:chilitag_origin_in_corner>
+      <xacro:chilitag_origin_in_corner name="chilitag${name_start + 1}" size="${size}" parent="${parent}">
+        <origin xyz="${offset_x}
+                     ${offset_y + offset_tag}
+                     ${offset_z}"
+                rpy="0 0 0"/>
+      </xacro:chilitag_origin_in_corner>
+      <xacro:chilitag_origin_in_corner name="chilitag${name_start + 2}" size="${size}" parent="${parent}">
+        <origin xyz="${offset_x + offset_tag}
+                     ${offset_y}
+                     ${offset_z}"
+                rpy="0 0 0"/>
+      </xacro:chilitag_origin_in_corner>
+      <xacro:chilitag_origin_in_corner name="chilitag${name_start + 3}" size="${size}" parent="${parent}">
+        <origin xyz="${offset_x + offset_tag}
+                     ${offset_y + offset_tag}
+                     ${offset_z}"
+                rpy="0 0 0"/>
+      </xacro:chilitag_origin_in_corner>
   </xacro:macro>
     <xacro:macro name="chilitag3d" params="name size parent *origin">

Commit message: Added macro for poi

File: urdf/chilitag.urdf.xacro (robot description, xacro)
@@ -100,4 +100,31 @@
       </xacro:chilitag_origin_in_corner>
   </xacro:macro>
+  <xacro:macro name="poi" params="name_start offset_tag size parent">
+      <xacro:property name="offset_set_1_x" value="0.6043" />
+      <xacro:property name="offset_set_1_y" value="-0.0857" />
+      <xacro:property name="offset_set_1_z" value="0.0002" />
+      <xacro:property name="offset_set_2_x" value="0.4043" />
+      <xacro:property name="offset_set_2_y" value="-0.5957" />
+      <xacro:property name="offset_set_2_z" value="0.0002" />
+      <xacro:property name="offset_set_3_x" value="-0.1057" />
+      <xacro:property name="offset_set_3_y" value="-0.7957" />
+      <xacro:property name="offset_set_3_z" value="0.0002" />
+      <xacro:property name="offset_set_4_x" value="0.4043" />
+      <xacro:property name="offset_set_4_y" value="0.4243" />
+      <xacro:property name="offset_set_4_z" value="0.0002" />
+      <xacro:property name="offset_set_5_x" value="-0.1057" />
+      <xacro:property name="offset_set_5_y" value="0.6243" />
+      <xacro:property name="offset_set_5_z" value="0.0002" />
+      <xacro:chilitag_4_set name_start="${name_start}" offset_x="${offset_set_1_x}" offset_y="${offset_set_1_y}" offset_z="${offset_set_1_z}" offset_tag="${offset_tag}" size="${size}" parent="${parent}">
+      </xacro:chilitag_4_set>
+      <xacro:chilitag_4_set name_start="${name_start + 4}" offset_x="${offset_set_2_x}" offset_y="${offset_set_2_y}" offset_z="${offset_set_2_z}" offset_tag="${offset_tag}" size="${size}" parent="${parent}">
+      </xacro:chilitag_4_set>
+      <xacro:chilitag_4_set name_start="${name_start + 8}" offset_x="${offset_set_3_x}" offset_y="${offset_set_3_y}" offset_z="${offset_set_3_z}" offset_tag="${offset_tag}" size="${size}" parent="${parent}">
+      </xacro:chilitag_4_set>
+      <xacro:chilitag_4_set name_start="${name_start + 12}" offset_x="${offset_set_4_x}" offset_y="${offset_set_4_y}" offset_z="${offset_set_4_z}" offset_tag="${offset_tag}" size="${size}" parent="${parent}">
+      </xacro:chilitag_4_set>
+      <xacro:chilitag_4_set name_start="${name_start + 16}" offset_x="${offset_set_5_x}" offset_y="${offset_set_5_y}" offset_z="${offset_set_5_z}" offset_tag="${offset_tag}" size="${size}" parent="${parent}">
+      </xacro:chilitag_4_set>
+  </xacro:macro>
     <xacro:macro name="chilitag3d" params="name size parent *origin">
     <joint name="${name}_joint" type="fixed">

Commit message: Added new chilitags for visualization in simulation and 9-er set of chilitags

File: urdf/chilitag.urdf.xacro (robot description, xacro)
@@ -100,4 +100,60 @@
       </xacro:chilitag_origin_in_corner>
   </xacro:macro>
+  <xacro:macro name="chilitag_9_set" params="name_start offset_x offset_y offset_z offset_tag size parent">
+      <xacro:chilitag_origin_in_corner name="chilitag${name_start}" size="${size}" parent="${parent}">
+        <origin xyz="${offset_x}
+                     ${offset_y}
+                     ${offset_z}"
+                rpy="0 0 0"/>
+      </xacro:chilitag_origin_in_corner>
+      <xacro:chilitag_origin_in_corner name="chilitag${name_start + 1}" size="${size}" parent="${parent}">
+        <origin xyz="${offset_x}
+                     ${offset_y + offset_tag}
+                     ${offset_z}"
+                rpy="0 0 0"/>
+      </xacro:chilitag_origin_in_corner>
+      <xacro:chilitag_origin_in_corner name="chilitag${name_start + 2}" size="${size}" parent="${parent}">
+        <origin xyz="${offset_x}
+                     ${offset_y + offset_tag * 2}
+                     ${offset_z}"
+                rpy="0 0 0"/>
+      </xacro:chilitag_origin_in_corner>
+      <xacro:chilitag_origin_in_corner name="chilitag${name_start + 3}" size="${size}" parent="${parent}">
+        <origin xyz="${offset_x + offset_tag}
+                     ${offset_y}
+                     ${offset_z}"
+                rpy="0 0 0"/>
+      </xacro:chilitag_origin_in_corner>
+      <xacro:chilitag_origin_in_corner name="chilitag${name_start + 4}" size="${size}" parent="${parent}">
+        <origin xyz="${offset_x + offset_tag}
+                     ${offset_y + offset_tag}
+                     ${offset_z}"
+                rpy="0 0 0"/>
+      </xacro:chilitag_origin_in_corner>
+      <xacro:chilitag_origin_in_corner name="chilitag${name_start + 5}" size="${size}" parent="${parent}">
+        <origin xyz="${offset_x + offset_tag}
+                     ${offset_y + offset_tag * 2}
+                     ${offset_z}"
+                rpy="0 0 0"/>
+      </xacro:chilitag_origin_in_corner>
+      <xacro:chilitag_origin_in_corner name="chilitag${name_start + 6}" size="${size}" parent="${parent}">
+        <origin xyz="${offset_x + offset_tag * 2}
+                     ${offset_y}
+                     ${offset_z}"
+                rpy="0 0 0"/>
+      </xacro:chilitag_origin_in_corner>
+      <xacro:chilitag_origin_in_corner name="chilitag${name_start + 7}" size="${size}" parent="${parent}">
+        <origin xyz="${offset_x + offset_tag * 2}
+                     ${offset_y + offset_tag}
+                     ${offset_z}"
+                rpy="0 0 0"/>
+      </xacro:chilitag_origin_in_corner>
+      <xacro:chilitag_origin_in_corner name="chilitag${name_start + 8}" size="${size}" parent="${parent}">
+        <origin xyz="${offset_x + offset_tag * 2}
+                     ${offset_y + offset_tag * 2}
+                     ${offset_z}"
+                rpy="0 0 0"/>
+      </xacro:chilitag_origin_in_corner>
+  </xacro:macro>
   <xacro:macro name="poi" params="name_start offset_tag size parent">
       <xacro:property name="offset_set_1_x" value="0.6043" />
@@ -116,14 +172,14 @@
       <xacro:property name="offset_set_5_y" value="0.6243" />
       <xacro:property name="offset_set_5_z" value="0.0002" />
-      <xacro:chilitag_4_set name_start="${name_start}" offset_x="${offset_set_1_x}" offset_y="${offset_set_1_y}" offset_z="${offset_set_1_z}" offset_tag="${offset_tag}" size="${size}" parent="${parent}">
-      </xacro:chilitag_4_set>
-      <xacro:chilitag_4_set name_start="${name_start + 4}" offset_x="${offset_set_2_x}" offset_y="${offset_set_2_y}" offset_z="${offset_set_2_z}" offset_tag="${offset_tag}" size="${size}" parent="${parent}">
-      </xacro:chilitag_4_set>
-      <xacro:chilitag_4_set name_start="${name_start + 8}" offset_x="${offset_set_3_x}" offset_y="${offset_set_3_y}" offset_z="${offset_set_3_z}" offset_tag="${offset_tag}" size="${size}" parent="${parent}">
-      </xacro:chilitag_4_set>
-      <xacro:chilitag_4_set name_start="${name_start + 12}" offset_x="${offset_set_4_x}" offset_y="${offset_set_4_y}" offset_z="${offset_set_4_z}" offset_tag="${offset_tag}" size="${size}" parent="${parent}">
-      </xacro:chilitag_4_set>
-      <xacro:chilitag_4_set name_start="${name_start + 16}" offset_x="${offset_set_5_x}" offset_y="${offset_set_5_y}" offset_z="${offset_set_5_z}" offset_tag="${offset_tag}" size="${size}" parent="${parent}">
-      </xacro:chilitag_4_set>
+      <xacro:chilitag_9_set name_start="${name_start}" offset_x="${offset_set_1_x}" offset_y="${offset_set_1_y}" offset_z="${offset_set_1_z}" offset_tag="${offset_tag}" size="${size}" parent="${parent}">
+      </xacro:chilitag_9_set>
+      <xacro:chilitag_9_set name_start="${name_start + 9}" offset_x="${offset_set_2_x}" offset_y="${offset_set_2_y}" offset_z="${offset_set_2_z}" offset_tag="${offset_tag}" size="${size}" parent="${parent}">
+      </xacro:chilitag_9_set>
+      <xacro:chilitag_9_set name_start="${name_start + 18}" offset_x="${offset_set_3_x}" offset_y="${offset_set_3_y}" offset_z="${offset_set_3_z}" offset_tag="${offset_tag}" size="${size}" parent="${parent}">
+      </xacro:chilitag_9_set>
+      <xacro:chilitag_9_set name_start="${name_start + 27}" offset_x="${offset_set_4_x}" offset_y="${offset_set_4_y}" offset_z="${offset_set_4_z}" offset_tag="${offset_tag}" size="${size}" parent="${parent}">
+      </xacro:chilitag_9_set>
+      <xacro:chilitag_9_set name_start="${name_start + 36}" offset_x="${offset_set_5_x}" offset_y="${offset_set_5_y}" offset_z="${offset_set_5_z}" offset_tag="${offset_tag}" size="${size}" parent="${parent}">
+      </xacro:chilitag_9_set>
   </xacro:macro>
     <xacro:macro name="chilitag3d" params="name size parent *origin">
