Commit message: Minor change to position of chilitags 9er

File: urdf/chilitag.urdf.xacro (robot description, xacro)
@@ -156,20 +156,26 @@
       </xacro:chilitag_origin_in_corner>
   </xacro:macro>
-  <xacro:macro name="poi" params="name_start offset_tag size parent">
-      <xacro:property name="offset_set_1_x" value="0.6043" />
-      <xacro:property name="offset_set_1_y" value="-0.0857" />
+  <xacro:macro name="bow" params="name_start offset_tag size parent">
+      <xacro:property name="offset_set_1_x" value="0.6105" />
+      <xacro:property name="offset_set_1_y" value="-0.0895" />
       <xacro:property name="offset_set_1_z" value="0.0002" />
-      <xacro:property name="offset_set_2_x" value="0.4043" />
-      <xacro:property name="offset_set_2_y" value="-0.5957" />
+      <xacro:property name="offset_set_2_x" value="0.4355" />
+      <xacro:property name="offset_set_2_y" value="0.4355" />
       <xacro:property name="offset_set_2_z" value="0.0002" />
-      <xacro:property name="offset_set_3_x" value="-0.1057" />
-      <xacro:property name="offset_set_3_y" value="-0.7957" />
+      <xacro:property name="offset_set_3_x" value="0.4355" />
+      <xacro:property name="offset_set_3_y" value="-0.6145" />
       <xacro:property name="offset_set_3_z" value="0.0002" />
-      <xacro:property name="offset_set_4_x" value="0.4043" />
-      <xacro:property name="offset_set_4_y" value="0.4243" />
+      <xacro:property name="offset_set_4_x" value="-0.0895" />
+      <xacro:property name="offset_set_4_y" value="0.6105" />
       <xacro:property name="offset_set_4_z" value="0.0002" />
-      <xacro:property name="offset_set_5_x" value="-0.1057" />
-      <xacro:property name="offset_set_5_y" value="0.6243" />
+      <xacro:property name="offset_set_5_x" value="-0.0895" />
+      <xacro:property name="offset_set_5_y" value="-0.7895" />
       <xacro:property name="offset_set_5_z" value="0.0002" />
+      <xacro:property name="offset_set_6_x" value="-0.6145" />
+      <xacro:property name="offset_set_6_y" value="0.4355" />
+      <xacro:property name="offset_set_6_z" value="0.0002" />
+      <xacro:property name="offset_set_7_x" value="-0.6145" />
+      <xacro:property name="offset_set_7_y" value="-0.6145" />
+      <xacro:property name="offset_set_7_z" value="0.0002" />
       <xacro:chilitag_9_set name_start="${name_start}" offset_x="${offset_set_1_x}" offset_y="${offset_set_1_y}" offset_z="${offset_set_1_z}" offset_tag="${offset_tag}" size="${size}" parent="${parent}">
       </xacro:chilitag_9_set>
@@ -181,4 +187,8 @@
       </xacro:chilitag_9_set>
       <xacro:chilitag_9_set name_start="${name_start + 36}" offset_x="${offset_set_5_x}" offset_y="${offset_set_5_y}" offset_z="${offset_set_5_z}" offset_tag="${offset_tag}" size="${size}" parent="${parent}">
+      </xacro:chilitag_9_set>
+      <xacro:chilitag_9_set name_start="${name_start + 45}" offset_x="${offset_set_6_x}" offset_y="${offset_set_6_y}" offset_z="${offset_set_6_z}" offset_tag="${offset_tag}" size="${size}" parent="${parent}">
+      </xacro:chilitag_9_set>
+      <xacro:chilitag_9_set name_start="${name_start + 54}" offset_x="${offset_set_7_x}" offset_y="${offset_set_7_y}" offset_z="${offset_set_7_z}" offset_tag="${offset_tag}" size="${size}" parent="${parent}">
       </xacro:chilitag_9_set>
   </xacro:macro>

Commit message: changed chilitag frame so x points right and y down similar to an image

File: urdf/chilitag.urdf.xacro (robot description, xacro)
@@ -33,5 +33,5 @@
       </inertial>
       <xacro:chilitag_visual_sized name="${name}" size="${size}">
-        <origin xyz="0 0 0" rpy="0 -1.57079632679 0"/>
+        <origin xyz="0 0 0" rpy="0 0 0"/>
       </xacro:chilitag_visual_sized>
       <!--
@@ -193,5 +193,5 @@
       </xacro:chilitag_9_set>
   </xacro:macro>
-    <xacro:macro name="chilitag3d" params="name size parent *origin">
+  <xacro:macro name="chilitag3d" params="name size parent *origin">
     <joint name="${name}_joint" type="fixed">
       <xacro:insert_block name="origin" />
@@ -206,5 +206,5 @@
       </inertial>
       <xacro:chilitag_visual_sized name="${name}" size="${size}">
-        <origin xyz="${size/2} ${size/2} 0" rpy="${-M_PI/2} ${M_PI/2} ${M_PI}"/>
+        <origin xyz="${size/2} ${size/2} 0" rpy="0 0 0"/>
       </xacro:chilitag_visual_sized>
     </link>

Commit message: Generalized z offset for bow

File: urdf/chilitag.urdf.xacro (robot description, xacro)
@@ -156,39 +156,32 @@
       </xacro:chilitag_origin_in_corner>
   </xacro:macro>
-  <xacro:macro name="bow" params="name_start offset_tag size parent">
+  <xacro:macro name="bow" params="name_start offset_tag offset_set_z size parent">
       <xacro:property name="offset_set_1_x" value="0.6105" />
       <xacro:property name="offset_set_1_y" value="-0.0895" />
-      <xacro:property name="offset_set_1_z" value="0.0002" />
       <xacro:property name="offset_set_2_x" value="0.4355" />
       <xacro:property name="offset_set_2_y" value="0.4355" />
-      <xacro:property name="offset_set_2_z" value="0.0002" />
       <xacro:property name="offset_set_3_x" value="0.4355" />
       <xacro:property name="offset_set_3_y" value="-0.6145" />
-      <xacro:property name="offset_set_3_z" value="0.0002" />
       <xacro:property name="offset_set_4_x" value="-0.0895" />
       <xacro:property name="offset_set_4_y" value="0.6105" />
-      <xacro:property name="offset_set_4_z" value="0.0002" />
       <xacro:property name="offset_set_5_x" value="-0.0895" />
       <xacro:property name="offset_set_5_y" value="-0.7895" />
-      <xacro:property name="offset_set_5_z" value="0.0002" />
       <xacro:property name="offset_set_6_x" value="-0.6145" />
       <xacro:property name="offset_set_6_y" value="0.4355" />
-      <xacro:property name="offset_set_6_z" value="0.0002" />
       <xacro:property name="offset_set_7_x" value="-0.6145" />
       <xacro:property name="offset_set_7_y" value="-0.6145" />
-      <xacro:property name="offset_set_7_z" value="0.0002" />
-      <xacro:chilitag_9_set name_start="${name_start}" offset_x="${offset_set_1_x}" offset_y="${offset_set_1_y}" offset_z="${offset_set_1_z}" offset_tag="${offset_tag}" size="${size}" parent="${parent}">
-      </xacro:chilitag_9_set>
-      <xacro:chilitag_9_set name_start="${name_start + 9}" offset_x="${offset_set_2_x}" offset_y="${offset_set_2_y}" offset_z="${offset_set_2_z}" offset_tag="${offset_tag}" size="${size}" parent="${parent}">
-      </xacro:chilitag_9_set>
-      <xacro:chilitag_9_set name_start="${name_start + 18}" offset_x="${offset_set_3_x}" offset_y="${offset_set_3_y}" offset_z="${offset_set_3_z}" offset_tag="${offset_tag}" size="${size}" parent="${parent}">
-      </xacro:chilitag_9_set>
-      <xacro:chilitag_9_set name_start="${name_start + 27}" offset_x="${offset_set_4_x}" offset_y="${offset_set_4_y}" offset_z="${offset_set_4_z}" offset_tag="${offset_tag}" size="${size}" parent="${parent}">
-      </xacro:chilitag_9_set>
-      <xacro:chilitag_9_set name_start="${name_start + 36}" offset_x="${offset_set_5_x}" offset_y="${offset_set_5_y}" offset_z="${offset_set_5_z}" offset_tag="${offset_tag}" size="${size}" parent="${parent}">
-      </xacro:chilitag_9_set>
-      <xacro:chilitag_9_set name_start="${name_start + 45}" offset_x="${offset_set_6_x}" offset_y="${offset_set_6_y}" offset_z="${offset_set_6_z}" offset_tag="${offset_tag}" size="${size}" parent="${parent}">
-      </xacro:chilitag_9_set>
-      <xacro:chilitag_9_set name_start="${name_start + 54}" offset_x="${offset_set_7_x}" offset_y="${offset_set_7_y}" offset_z="${offset_set_7_z}" offset_tag="${offset_tag}" size="${size}" parent="${parent}">
+      <xacro:chilitag_9_set name_start="${name_start}" offset_x="${offset_set_1_x}" offset_y="${offset_set_1_y}" offset_z="${offset_set_z}" offset_tag="${offset_tag}" size="${size}" parent="${parent}">
+      </xacro:chilitag_9_set>
+      <xacro:chilitag_9_set name_start="${name_start + 9}" offset_x="${offset_set_2_x}" offset_y="${offset_set_2_y}" offset_z="${offset_set_z}" offset_tag="${offset_tag}" size="${size}" parent="${parent}">
+      </xacro:chilitag_9_set>
+      <xacro:chilitag_9_set name_start="${name_start + 18}" offset_x="${offset_set_3_x}" offset_y="${offset_set_3_y}" offset_z="${offset_set_z}" offset_tag="${offset_tag}" size="${size}" parent="${parent}">
+      </xacro:chilitag_9_set>
+      <xacro:chilitag_9_set name_start="${name_start + 27}" offset_x="${offset_set_4_x}" offset_y="${offset_set_4_y}" offset_z="${offset_set_z}" offset_tag="${offset_tag}" size="${size}" parent="${parent}">
+      </xacro:chilitag_9_set>
+      <xacro:chilitag_9_set name_start="${name_start + 36}" offset_x="${offset_set_5_x}" offset_y="${offset_set_5_y}" offset_z="${offset_set_z}" offset_tag="${offset_tag}" size="${size}" parent="${parent}">
+      </xacro:chilitag_9_set>
+      <xacro:chilitag_9_set name_start="${name_start + 45}" offset_x="${offset_set_6_x}" offset_y="${offset_set_6_y}" offset_z="${offset_set_z}" offset_tag="${offset_tag}" size="${size}" parent="${parent}">
+      </xacro:chilitag_9_set>
+      <xacro:chilitag_9_set name_start="${name_start + 54}" offset_x="${offset_set_7_x}" offset_y="${offset_set_7_y}" offset_z="${offset_set_z}" offset_tag="${offset_tag}" size="${size}" parent="${parent}">
       </xacro:chilitag_9_set>
   </xacro:macro>

Commit message: Added bow 6:00 config

File: urdf/chilitag.urdf.xacro (robot description, xacro)
@@ -171,4 +171,6 @@
       <xacro:property name="offset_set_7_x" value="-0.6145" />
       <xacro:property name="offset_set_7_y" value="-0.6145" />
+      <xacro:property name="offset_set_8_x" value="-0.7895" />
+      <xacro:property name="offset_set_8_y" value="-0.0895" />
       <xacro:chilitag_9_set name_start="${name_start}" offset_x="${offset_set_1_x}" offset_y="${offset_set_1_y}" offset_z="${offset_set_z}" offset_tag="${offset_tag}" size="${size}" parent="${parent}">
       </xacro:chilitag_9_set>
@@ -184,4 +186,6 @@
       </xacro:chilitag_9_set>
       <xacro:chilitag_9_set name_start="${name_start + 54}" offset_x="${offset_set_7_x}" offset_y="${offset_set_7_y}" offset_z="${offset_set_z}" offset_tag="${offset_tag}" size="${size}" parent="${parent}">
+      </xacro:chilitag_9_set>
+      <xacro:chilitag_9_set name_start="${name_start - 9}" offset_x="${offset_set_8_x}" offset_y="${offset_set_8_y}" offset_z="${offset_set_z}" offset_tag="${offset_tag}" size="${size}" parent="${parent}">
       </xacro:chilitag_9_set>
   </xacro:macro>
